File: schematic/CrashButtonESP8266D1.brd (EAGLE design)
At the start: 101 x 101.6 mm, 32 parts, among them U1 ESP12E_DEVKIT

Commit message: added board that uses D1 mini style esp8266
Parts:
- removed U1: ESP12E_DEVKIT, ESP12E_DEVKIT:ESP12E_DEVKIT
- added WEMOS1: ESP8266, esp8266modules:WEMOS-D1-MINI
- R1: value 470 -> 220
- moved D1 73.8 mm to (0.00, -38.4)
- moved C1 73.5 mm to (0.00, -41.0)
- moved C10 71.8 mm to (41.3, 0.00)
- moved C11 71.8 mm to (35.7, -20.6)
- moved C12 71.8 mm to (20.6, -35.7)
- moved C13 71.8 mm to (30.5, -12.7)
- moved C14 71.8 mm to (17.1, -10.2)
- moved C2 71.8 mm to (-20.6, -35.7)
- moved C3 71.8 mm to (-35.7, -20.6)
- moved C4 71.8 mm to (-41.3, 0.00)
- moved C5 71.8 mm to (-35.7, 20.6)
- moved C6 71.8 mm to (-20.6, 35.7)
- moved C7 71.8 mm to (0.00, 41.3)
- moved C8 71.8 mm to (20.6, 35.7)
- moved C9 71.8 mm to (35.7, 20.6)
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Connections:
- net LEDDIN renamed N$10
- net VCC renamed N$11
- removed net N$10 (its old number): S1.1, S2.1, U1.D2
- new net BUTTON: S1.1, S2.1, WEMOS1.D2
- new net LEDDATOUT: LED12.2-DOUT
- net GND: now also WEMOS1.GND; no longer U1.GND@1
- net LEDDINRAW: now also WEMOS1.D4; no longer U1.D4
- net VIN: now also WEMOS1.5V; no longer U1.VIN
Routing:
- net BUTTON: track 0.00 -> 97.7 mm
- net N$10 (its old number): track 93.4 -> 0.00 mm
- net LEDDINRAW: track 63.3 -> 53.4 mm
- net VIN: track 322.3 -> 332.3 mm
- net N$11: track 9.04 -> 6.13 mm
- net N$10: track 20.0 -> 20.6 mm
Other:
- board text added: "v20161229"
- board text removed: "v20161222"

Commit message: schematic updates
Parts:
- added J2: (no value), SparkFun-Connectors:1X02
- added R2: 220, SparkFun-Resistors:0603
Connections:
- new net N$14: R2.2, WEMOS1.D2
- net BUTTON: now also J2.1, R2.1; no longer WEMOS1.D2
- net GND: now also J2.2
Routing:
- net N$14: track 0.00 -> 12.7 mm
- net BUTTON: track 97.7 -> 89.3 mm
Other:
- board text added: "button"
- board text added: "v20170102"
- board text added: "ws2812"
- board text removed: "NodeMCU ESP8266 on back"
- board text removed: "v20161229"
Changed lines of the file:
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@@
 <wire x1="-77.47" y1="50.8" x2="50.8" y2="50.8" width="0.0254" layer="48" style="longdash"/>
 <wire x1="50.8" y1="50.8" x2="73.66" y2="50.8" width="0.0254" layer="48" style="longdash"/>
-<text x="-11.43" y="34.29" size="1.778" layer="25">CrashButtonESP</text>
-<text x="-7.62" y="-21.59" size="1.778" layer="25">todbot.com</text>
-<text x="-7.62" y="-24.13" size="1.778" layer="25">v20161229</text>
+<text x="-11.43" y="33.02" size="1.778" layer="25">CrashButtonESP</text>
+<text x="-7.62" y="-17.78" size="1.778" layer="25">todbot.com</text>
+<text x="-7.62" y="-20.32" size="1.778" layer="25">v20170102</text>
 <wire x1="-81.28" y1="-20.32" x2="69.85" y2="-20.32" width="0.0254" layer="48" style="longdash"/>
 <hole x="20.32" y="20.32" drill="3.7973"/>
@@
 <wire x1="50.8" y1="-50.165" x2="50.8" y2="-52.07" width="0.0254" layer="48" style="longdash"/>
 <wire x1="-20.32" y1="54.61" x2="-20.32" y2="-57.15" width="0.0254" layer="48" style="longdash"/>
-<text x="1.27" y="-11.43" size="1.778" layer="25" rot="R90">NodeMCU ESP8266 on back</text>
-<text x="-16.51" y="-23.495" size="1.27" layer="25">gnd</text>
-<text x="-19.05" y="-26.035" size="1.27" layer="25">leddat</text>
-<text x="-16.51" y="-28.575" size="1.27" layer="25">+5V</text>
-<text x="-16.51" y="-28.575" size="1.27" layer="25">+5V</text>
+<text x="-13.462" y="-22.225" size="1.27" layer="25" rot="R180">gnd</text>
+<text x="-13.462" y="-24.765" size="1.27" layer="25" rot="R180">leddat</text>
+<text x="-13.462" y="-27.305" size="1.27" layer="25" rot="R180">+5V</text>
 <wire x1="-22.86" y1="54.61" x2="-22.86" y2="-57.15" width="0.0254" layer="48" style="longdash"/>
 <wire x1="22.86" y1="52.705" x2="22.86" y2="-59.055" width="0.0254" layer="48" style="longdash"/>
 <wire x1="-63.5" y1="-50.546" x2="73.66" y2="-50.546" width="0" layer="48" style="shortdash"/>
+<text x="-7.62" y="-29.845" size="1.27" layer="25" rot="R180">ws2812</text>
+<text x="24.638" y="25.019" size="1.27" layer="25">gnd</text>
+<text x="24.638" y="27.559" size="1.27" layer="25">button</text>
+<polygon width="0.254" layer="41">
+<vertex x="-8.382" y="24.13"/>
+<vertex x="-8.382" y="17.018"/>
+<vertex x="8.382" y="17.018"/>
+<vertex x="8.382" y="24.13"/>
+</polygon>
 </plain>
 <attributes>
@@
 </element>
 <element name="WEMOS1" library="esp8266modules" package="WEMOS-D1-MINI" value="ESP8266" x="-1.27" y="7.62"/>
+<element name="R2" library="SparkFun-Resistors" package="0603" value="220" x="22.86" y="11.43" rot="R270">
+<attribute name="PROD_ID" value="RES-07869" x="22.86" y="11.43" size="1.778" layer="27" rot="R270" display="off"/>
+</element>
+<element name="J2" library="SparkFun-Connectors" package="1X02" value="" x="22.86" y="27.94" smashed="yes" rot="R270">
+<attribute name="NAME" x="22.352" y="29.845" size="0.6096" layer="25" font="vector" ratio="20"/>
+<attribute name="VALUE" x="20.828" y="29.21" size="0.6096" layer="27" font="vector" ratio="20" rot="R270"/>
+</element>
 </elements>
 <signals>
@@
 <contactref element="J1" pad="1"/>
 <contactref element="WEMOS1" pad="GND"/>
+<contactref element="J2" pad="2"/>
 </signal>
 <signal name="N$1">
@@
 <contactref element="LED11" pad="4-DIN"/>
 <wire x1="39.39074375" y1="-19.9132375" x2="47.37" y2="-2.45" width="0.4064" layer="1"/>
-</signal>
-<signal name="BUTTON">
-<contactref element="S1" pad="1"/>
-<contactref element="S2" pad="1"/>
-<wire x1="12.7" y1="33.02" x2="0" y2="33.02" width="0.4064" layer="1"/>
-<wire x1="-7.62" y1="33.02" x2="0" y2="33.02" width="0.4064" layer="1"/>
-<wire x1="-7.62" y1="33.02" x2="-12.7" y2="33.02" width="0.4064" layer="1"/>
-<wire x1="-12.7" y1="33.02" x2="-15.24" y2="30.48" width="0.4064" layer="1"/>
-<wire x1="-15.24" y1="30.48" x2="-15.24" y2="19.05" width="0.4064" layer="1"/>
-<wire x1="-15.24" y1="19.05" x2="-15.24" y2="11.37" width="0.4064" layer="1"/>
-<wire x1="-15.24" y1="11.37" x2="-20.36" y2="6.25" width="0.4064" layer="1"/>
-<wire x1="25.36" y1="6.25" x2="25.36" y2="6.39" width="0.4064" layer="1"/>
-<wire x1="25.36" y1="6.39" x2="20.32" y2="11.43" width="0.4064" layer="1"/>
-<wire x1="20.32" y1="11.43" x2="16.51" y2="11.43" width="0.4064" layer="1"/>
-<wire x1="16.51" y1="11.43" x2="15.24" y2="12.7" width="0.4064" layer="1"/>
-<wire x1="15.24" y1="12.7" x2="15.24" y2="30.48" width="0.4064" layer="1"/>
-<wire x1="15.24" y1="30.48" x2="12.7" y2="33.02" width="0.4064" layer="1"/>
-<contactref element="WEMOS1" pad="D2"/>
-<wire x1="11.43" y1="7.62" x2="15.24" y2="7.62" width="0.4064" layer="1"/>
-<wire x1="15.24" y1="7.62" x2="16.51" y2="8.89" width="0.4064" layer="1"/>
-<wire x1="16.51" y1="8.89" x2="16.51" y2="11.43" width="0.4064" layer="1"/>
 </signal>
 <signal name="N$12">
@@
 <wire x1="38.1" y1="0" x2="41.275" y2="-0.85" width="0.4064" layer="1"/>
 <wire x1="36.170190625" y1="19.901378125" x2="33.02" y2="20.32" width="0.4064" layer="1"/>
-<wire x1="33.02" y1="20.32" x2="24.156759375" y2="36.94074375" width="0.4064" layer="1"/>
+<wire x1="33.02" y1="20.32" x2="29.539946875" y2="26.84595" width="0.4064" layer="1"/>
+<wire x1="29.539946875" y1="26.84595" x2="28.7314625" y2="28.36205625" width="0.4064" layer="1"/>
+<wire x1="28.7314625" y1="28.36205625" x2="27.922975" y2="29.878165625" width="0.4064" layer="1"/>
+<wire x1="27.922975" y1="29.878165625" x2="24.156759375" y2="36.94074375" width="0.4064" layer="1"/>
 <wire x1="21.37361875" y1="35.320190625" x2="19.05" y2="34.29" width="0.4064" layer="1"/>
 <wire x1="19.05" y1="34.29" x2="2.45" y2="44.07" width="0.4064" layer="1"/>
@@
 <wire x1="-1.15" y1="-38.735" x2="-0.85" y2="-41.021" width="0.4064" layer="1"/>
 </signal>
+<signal name="BUTTON">
+<contactref element="R2" pad="1"/>
+<contactref element="S2" pad="1"/>
+<contactref element="S1" pad="1"/>
+<wire x1="-20.36" y1="6.25" x2="-20.36" y2="8.85" width="0.4064" layer="1"/>
+<wire x1="-20.36" y1="8.85" x2="-17.78" y2="11.43" width="0.4064" layer="1"/>
+<wire x1="-17.78" y1="11.43" x2="-16.51" y2="12.7" width="0.4064" layer="1"/>
+<wire x1="-16.51" y1="12.7" x2="-16.51" y2="24.13" width="0.4064" layer="1"/>
+<wire x1="-16.51" y1="24.13" x2="-12.7" y2="27.94" width="0.4064" layer="1"/>
+<wire x1="-12.7" y1="27.94" x2="-10.16" y2="27.94" width="0.4064" layer="1"/>
+<wire x1="-10.16" y1="27.94" x2="13.97" y2="27.94" width="0.4064" layer="1"/>
+<wire x1="13.97" y1="27.94" x2="16.51" y2="25.4" width="0.4064" layer="1"/>
+<wire x1="16.51" y1="25.4" x2="16.51" y2="15.24" width="0.4064" layer="1"/>
+<wire x1="20.32" y1="26.67" x2="19.05" y2="25.4" width="0.4064" layer="1"/>
+<wire x1="19.05" y1="25.4" x2="16.51" y2="25.4" width="0.4064" layer="1"/>
+<wire x1="25.654" y1="9.652" x2="25.654" y2="6.544" width="0.4064" layer="1"/>
+<wire x1="25.654" y1="6.544" x2="25.36" y2="6.25" width="0.4064" layer="1"/>
+<wire x1="20.32" y1="26.67" x2="21.59" y2="27.94" width="0.4064" layer="1"/>
+<wire x1="22.86" y1="12.28" x2="24.55" y2="12.28" width="0.4064" layer="1"/>
+<wire x1="24.55" y1="12.28" x2="25.4" y2="11.43" width="0.4064" layer="1"/>
+<wire x1="25.4" y1="11.43" x2="25.654" y2="11.176" width="0.4064" layer="1"/>
+<wire x1="25.654" y1="11.176" x2="25.654" y2="9.652" width="0.4064" layer="1"/>
+<wire x1="22.86" y1="12.28" x2="22.86" y2="13.462" width="0.4064" layer="1"/>
+<wire x1="22.86" y1="13.462" x2="21.844" y2="14.478" width="0.4064" layer="1"/>
+<wire x1="21.844" y1="14.478" x2="17.272" y2="14.478" width="0.4064" layer="1"/>
+<wire x1="17.272" y1="14.478" x2="16.51" y2="15.24" width="0.4064" layer="1"/>
+<contactref element="J2" pad="1"/>
+<wire x1="22.86" y1="27.94" x2="21.59" y2="27.94" width="0.4064" layer="1"/>
+</signal>
+<signal name="N$14">
+<contactref element="WEMOS1" pad="D2"/>
+<contactref element="R2" pad="2"/>
+<wire x1="11.43" y1="7.62" x2="15.24" y2="7.62" width="0.4064" layer="1"/>
+<wire x1="15.24" y1="7.62" x2="17.78" y2="10.16" width="0.4064" layer="1"/>
+<wire x1="22.86" y1="10.58" x2="18.2" y2="10.58" width="0.4064" layer="1"/>
+<wire x1="18.2" y1="10.58" x2="17.78" y2="10.16" width="0.4064" layer="1"/>
+</signal>
 </signals>

Commit message: updated schematic
Parts:
- R2: value 220 -> 1k
Changed lines of the file:
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@@
+<vertex x="8.382" y="24.13"/>
+</polygon>
+<polygon width="0.254" layer="42">
+<vertex x="-8.382" y="24.13"/>
+<vertex x="-8.382" y="17.018"/>
+<vertex x="8.382" y="17.018"/>
 <vertex x="8.382" y="24.13"/>
 </polygon>
@@
 </element>
 <element name="WEMOS1" library="esp8266modules" package="WEMOS-D1-MINI" value="ESP8266" x="-1.27" y="7.62"/>
-<element name="R2" library="SparkFun-Resistors" package="0603" value="220" x="22.86" y="11.43" rot="R270">
+<element name="R2" library="SparkFun-Resistors" package="0603" value="1k" x="22.86" y="11.43" rot="R270">
 <attribute name="PROD_ID" value="RES-07869" x="22.86" y="11.43" size="1.778" layer="27" rot="R270" display="off"/>
 </element>
